File: BrainFM.sch (KiCad schematic (older format))
At the start: 15 parts, among them J1 USB_B_Micro, U1 PAM8302AAD, U2 MCP73831-2-OT, U3 TLV75801PDBV

Commit message: work on PCM5012
Parts:
- added C?: .1 uf, symbol Device:C
- added C?: 10 uf, symbol Device:CP1
- added C? (x2): 2.2 uf, symbol Device:C
- added C? (x2): 2.2 nf, symbol Device:C
- added LS1: Speaker, symbol Device:Speaker
- added R? (x2): 470, Resistor_SMD:R_0805_2012Metric_Pad1.20x1.40mm_HandSolder, symbol Device:R
- added U4: ESP32-WROOM-32, RF_Module:ESP32-WROOM-32, symbol RF_Module:ESP32-WROOM-32
- added U5: PCM5102, Package_SO:TSSOP-20_4.4x6.5mm_P0.65mm, symbol Audio:PCM5102
- C1, C2, C3, C4, C5: footprint Capacitor_SMD:C_0805_2012Metric_Pad1.15x1.40mm_HandSolder -> Capacitor_SMD:C_0805_2012Metric_Pad1.18x1.45mm_HandSolder
- J1: symbol Connector:USB_B_Micro -> BrainFM-rescue:USB_B_Micro-Connector
- R1, R2: footprint Resistor_SMD:R_0805_2012Metric_Pad1.15x1.40mm_HandSolder -> Resistor_SMD:R_0805_2012Metric_Pad1.20x1.40mm_HandSolder
- R3: value R -> 10k; footprint Resistor_SMD:R_0805_2012Metric_Pad1.15x1.40mm_HandSolder -> Resistor_SMD:R_0805_2012Metric_Pad1.20x1.40mm_HandSolder
- R4: value R -> 2k; footprint Resistor_SMD:R_0805_2012Metric_Pad1.15x1.40mm_HandSolder -> Resistor_SMD:R_0805_2012Metric_Pad1.20x1.40mm_HandSolder
Connections:
- net labels added: LEFT, RIGHT
- wire segments 63 -> 118

Commit message: update schematic and layout
Parts:
- added C10, C16, C8: 10 uf, symbol Device:CP1
- added C11, C9: .1 uf, Capacitor_SMD:C_0805_2012Metric_Pad1.18x1.45mm_HandSolder, symbol Device:C
- added C14: 0.1 uf, Capacitor_SMD:C_0805_2012Metric_Pad1.18x1.45mm_HandSolder, symbol Device:C
- C12, C13, C15, C17, C7: renamed from C?; footprint (none) -> Capacitor_SMD:C_0805_2012Metric_Pad1.18x1.45mm_HandSolder
- gave numbers to parts that had none: 3
Connections:
- wire segments 118 -> 157
Other:
- moved on the sheet: C13, C15, C17
