File: BrainFM_MAX98357/BrainFM_MAX98357_PROTO.kicad_pcb (KiCad board)
At the start: 2 copper layers, 28.5 x 51.8 mm, 16 parts, among them J1 USB_B_Micro, J2 Conn_01x07_Male, U2 MCP73831-2-OT, U3 TLV75801PDBV, U4 ESP32-WROOM-32

Commit message: change TLV75801 for TC1262
Parts:
- removed R3: 10k, Resistor_SMD:R_0805_2012Metric_Pad1.20x1.40mm_HandSolder
- removed R4: 2k, Resistor_SMD:R_0805_2012Metric_Pad1.20x1.40mm_HandSolder
- removed REF** (x2): PinHeader_1x02_P2.54mm_Vertical, Connector_PinHeader_2.54mm:PinHeader_1x02_P2.54mm_Vertical
- U3: value TLV75801PDBV -> TC1262-33; footprint Package_TO_SOT_SMD:SOT-23-5 -> Package_TO_SOT_SMD:SOT-223
- moved C5 11.4 mm to (142.5, 83.0), turned to 270 degrees
- moved C4 5.70 mm to (142.5, 96.9)
- moved U3 1.39 mm to (145.7, 90.2)
Connections:
- C5 pad 1: +3V3 -> -BATT
- C5 pad 2: -BATT -> +3V3
- U3 pad 3: VCC -> +3V3
- U3 pad 4: Net-(R3-Pad2) -> (no net)
Routing:
- net +3V3: track 63.4 -> 31.8 mm
- net VCC: track 25.4 -> 3.74 mm
- net Net-(R3-Pad2): track 5.57 -> 0.00 mm
- removed copper zone on B.Cu, net -BATT
- removed copper zone on F.Cu, net -BATT

Commit message: drc runs clean
Parts:
- added REF**: PinHeader_1x02_P2.54mm_Vertical, Connector_PinHeader_2.54mm:PinHeader_1x02_P2.54mm_Vertical, F.Cu at (156.8, 66.0)
- added REF**: PinHeader_1x02_P2.54mm_Vertical, Connector_PinHeader_2.54mm:PinHeader_1x02_P2.54mm_Vertical, F.Cu at (154.5, 86.0)
Routing:
- net VCC: track 3.74 -> 22.8 mm
- net +3V3: track 31.8 -> 47.0 mm
- net -BATT: track 29.8 -> 32.4 mm
- added copper zone on B.Cu, net -BATT
- added copper zone on F.Cu, net -BATT

Commit message: sent to osh park
Parts:
- removed the REF** at (156.8, 66.0)
- removed the REF** at (154.5, 86.0)
- added COM: PinHeader_1x02_P2.54mm_Vertical, Connector_PinHeader_2.54mm:PinHeader_1x02_P2.54mm_Vertical, F.Cu at (157.0, 65.8)
- added POW: PinHeader_1x02_P2.54mm_Vertical, Connector_PinHeader_2.54mm:PinHeader_1x02_P2.54mm_Vertical, F.Cu at (154.5, 83.5)
- added R3: 10k, Resistor_SMD:R_0805_2012Metric_Pad1.20x1.40mm_HandSolder, B.Cu at (133.8, 71.5)
- added REF**: OSHW-Symbol_6.7x6mm_SilkScreen, Symbol:OSHW-Symbol_6.7x6mm_SilkScreen, B.Cu at (155.5, 54.0)
- added SW1: SW_SPDT_CK-JS102011SAQN, Button_Switch_SMD:SW_SPDT_CK-JS102011SAQN, F.Cu at (154.5, 94.8)
- moved C1 3.50 mm to (145.1, 86.4)
- moved C2 3.50 mm to (141.0, 85.1)
- moved D1 3.50 mm to (144.1, 94.0)
- moved J1 3.50 mm to (141.3, 99.1)
- moved R1 3.50 mm to (137.5, 92.4)
- moved R2 3.50 mm to (146.4, 90.2)
- moved U2 3.50 mm to (141.3, 90.2)
Connections:
- J2 pad 4: GAIN -> Net-(J2-Pad4)
Routing:
- net Net-(J2-Pad4): track 0.00 -> 22.7 mm
- net Net-(C1-Pad1): track 3.46 -> 14.0 mm
- net +3V3: track 47.0 -> 55.4 mm
- net VCC: track 22.8 -> 24.4 mm, vias 0 -> 1
Other:
- board text added: "+"
- board text added: "-"
- board text added: "BrainFM_MAX98357_PROTO V1"
- board text added: "TX"
